Commit message: here the new file robot_core_2 is used for the structure of the bot

File: description/robot_core_2.xacro (robot description, xacro)
@@ -2,21 +2,4 @@
 <robot xmlns:xacro="http://www.ros.org/wiki/xacro" name ="robot">
     <xacro:include filename="inertial_macros.xacro"/>
-    <xacro:property name="chassis_length" value="0.444"/>
-    <xacro:property name="chassis_width" value="0.444"/>
-    <xacro:property name="chassis_height" value="0.152"/>
-    <xacro:property name="chassis_mass" value="1.0"/>
-    <!-- as there are two wheels but here common parameters are defined -->
-    <xacro:property name="wheel_radius" value="0.076"/>
-    <xacro:property name="wheel_thickness" value="0.076"/>
-    <xacro:property name="wheel_mass" value="0.05"/>
-    <xacro:property name="wheel_offset_x" value="0.226"/>
-    <xacro:property name="wheel_offset_y" value="0.1485"/>
-    <xacro:property name="wheel_offset_z" value="0.01"/>
-    <!-- there are two caster wheels but common parameters are defined    -->
-    <xacro:property name="caster_wheel_radius" value="0.08"/>
-    <xacro:property name="caster_wheel_mass" value="0.01"/>
-    <xacro:property name="caster_wheel_offset_x" value="0.075"/>
-    <xacro:property name="caster_wheel_offset_z" value="${0.101 - 0.08 + 0.08}"/>
-<!-- need to be check the above -->
     <!-- robot apearence -->
     <material name="white">
@@ -37,12 +20,4 @@
  <!-- BASE LINK -->
     <link name="base_link">
-    </link>
-<!-- BASE_FOOTPRINT LINK -->
-    <joint name="base_footprint_joint" type="fixed">
-        <parent link="base_link"/>
-        <child link="base_footprint"/>
-        <origin xyz="0 0 0" rpy="0 0 0"/>
-    </joint>
-    <link name="base_footprint">
     </link>
  <!-- CHASSIS LINK -->

Commit message: changes in origin

File: description/robot_core_2.xacro (robot description, xacro)
@@ -25,16 +25,16 @@
         <parent link="base_link"/>
         <child link="chassis"/>
-        <origin xyz="-0.1 0 0"/> <!--<origin xyz="${-wheel_offset_x} 0 ${-wheel_offset_z}"/>--><!-- here the origin is set just behind the mid of chessi-->
+        <origin xyz="-0.1 0 0"/>
     </joint>
     <link name="chassis">
         <visual>
-            <origin xyz="0.22 0 0.075"/>
+            <origin xyz="0.22 0 0.076"/>
             <geometry>
                 <box size="0.44 0.44 0.15"/><!-- <box size="${chassis_length} ${chassis_width} ${chassis_height}"/> -->
             </geometry>
-            <material name="orange"/>
+            <material name="red"/>
         </visual>
         <collision>
-            <origin xyz="0.22 0 0.075"/>
+            <origin xyz="0.22 0 0.076"/>
             <geometry>
                 <box size="0.44 0.44 0.15"/>
@@ -42,9 +42,9 @@
         </collision>
         <xacro:inertial_box mass="0.5" x="0.44" y="0.44" z="0.15"><!-- <xacro:inertial_box mass="0.5" x="${chassis_length}" y="${chassis_width}" z="${chassis_height}"> -->
-             <origin xyz="0.22 0 0.075" rpy="0 0 0"/><!--<origin xyz="${chassis_length/2} 0 ${chassis_height/2}" rpy="0 0 0"/> -->
+             <origin xyz="0.22 0 0.076" rpy="0 0 0"/><!--<origin xyz="${chassis_length/2} 0 ${chassis_height/2}" rpy="0 0 0"/> -->
         </xacro:inertial_box>
     </link>
     <gazebo reference="chassis">
-        <material>Gazebo/Orange</material>
+        <material>Gazebo/Red</material>
     </gazebo>
     <!-- LEFT WHEEL LINK -->
@@ -52,5 +52,5 @@
         <parent link="base_link"/>
         <child link="left_wheel"/>
-        <origin xyz="0 0.175 0" rpy="-${pi/2} 0 0" />
+        <origin xyz="0 0.222 0" rpy="-${pi/2} 0 0" />
         <axis xyz="0 0 1"/>
     </joint>
@@ -60,5 +60,5 @@
                 <cylinder radius="0.08" length="0.08"/><!-- <cylinder radius="${wheel_radius}" length="${wheel_thickness}"/>/-->
             </geometry>
-            <material name="blue"/>
+            <material name= "blue"/>
         </visual>
         <collision>
@@ -78,5 +78,5 @@
         <parent link="base_link"/>
         <child link="right_wheel"/>
-        <origin xyz="0 -0.175 0" rpy="${pi/2} 0 0" />
+        <origin xyz="0 -0.222 0" rpy="${pi/2} 0 0" />
         <axis xyz="0 0 -1"/>
     </joint>
